File: 3_Nav.kicad_sch (KiCad schematic)
At the start: 59 parts, among them J401 GNSS, J402 Conn_Coaxial, Q401 Q_NMOS, SW401 SW_Push, SW402 SW_Push, U401 LPS22HH, U402 MS5607, U403 STM32F446VETx, U404 ICM-42688-P, U405 LSM6DSO32TR, U406 W25Q128JVE, U407 THD-2528-11SD-GF, U408 Ra-08H, Y401 YXC YSX321SL

Commit message: Continued connections for the new NAV
Added continuity sensing through a 8:1 mux
Restructured schematic so that everything actually fits in page 4
Updated CubeMX (ioc) file with pinout
Parts:
- removed C401, C402, C410, C411, C413, C422, C423: 100n, Capacitor_SMD:C_0603_1608Metric, symbol Device:C
- removed C412: 10n, Capacitor_SMD:C_0603_1608Metric, symbol Device:C
- removed C414: 2u2, Capacitor_SMD:C_0603_1608Metric, symbol Device:C
- removed C421: 10u, Capacitor_SMD:C_0805_2012Metric, symbol Device:C
- removed C424: 47u, Capacitor_SMD:C_0805_2012Metric, symbol Device:C
- removed D405: D_TVS, LED_SMD:LED_0603_1608Metric, symbol Device:D_TVS
- removed J402: Conn_Coaxial, Connector_Coaxial:SMA_Molex_73251-2200_Horizontal, symbol Connector:Conn_Coaxial
- removed R403, R404, R405, R406: 4k7, Resistor_SMD:R_0603_1608Metric, symbol Device:R
- removed R415: 10k, Resistor_SMD:R_0603_1608Metric, symbol Device:R
- removed R416: 810k, Resistor_SMD:R_0603_1608Metric, symbol Device:R
- removed U401: LPS22HH, Polaris:LPS22HH, symbol Sensor_Pressure:LPS22HH
- removed U402: MS5607, Package_LGA:LGA-8_3x5mm_P1.25mm, symbol Sensor_Pressure:MS5607-02BA
- removed U404: ICM-42688-P, Polaris:ICM-42688-P, symbol Polaris_symbols:ICM-42688-P
- removed U405: LSM6DSO32TR, Polaris:LSM6DSO32TR, symbol Polaris_symbols:LSM6DSO32TR
- removed U407: THD-2528-11SD-GF, Polaris:TF-SMD_THD2528-11SD-GF, symbol Polaris_symbols:MicroSD_THD2528-11SD-GF
- removed U408: Ra-08H, Polaris:RA-08H, symbol Polaris_symbols:Ai-Thinker_Ra-08H
- added C405: 1u, symbol Device:C
- added C406: 100n, symbol Device:C
- added C408, C409: 2u2, symbol Device:C
- R407: renamed from R401; now left out of the parts list
- renumbered C416 to C403, C415 to C404, C419 to C407, C409 to C410, C408 to C411, C420 to C412, C407 to C413, C406 to C414, C405 to C415, C404 to C416, C403 to C417, C417 to C418, C418 to C419, D403 to D401, D401 to D402, D402 to D403, R408 to R405, R407 to R406, R409 to R408, R410 to R409, R411 to R413, R413 to R414, R414 to R415, U406 to U404
Connections:
- net GND: now also C405.2, C406.2, C408.2, C409.2
- net ~{MUX_EN}: now reaches U403.15 (PC0)
- net at U403.21 (VREF+): now also C405.1, C406.1
- net PYRO_SENSE: now reaches U403.25 (PA2)
- net at U403.48 (VCAP_1): now also C408.1
- net at U403.73 (VCAP_2): now also C409.1
- net PB3: now reaches U403.89 (PB3)
- net PB4: now reaches U403.90 (PB4)
- net PB5: now reaches U403.91 (PB5)
- net DROGUE_S0 renamed PYRO_2
- net DROGUE_S1 renamed PYRO_3
- net FIRE_S0 renamed PYRO_0
- net FIRE_S1 renamed PYRO_1
- net MAIN_S0 renamed PYRO_4
- net MAIN_S1 renamed PYRO_5
- net PC13 renamed MUX_A
- net PC14 renamed MUX_B
- net PC15 renamed MUX_C
Other:
- added sheet 3_1_IMU0 (3_1_IMU0.kicad_sch)
- added sheet 3_2_IMU1 (3_2_IMU1.kicad_sch)
- added sheet 3_3_BARO0 (3_3_BARO0.kicad_sch)
- added sheet 3_4_BARO1 (3_4_BARO1.kicad_sch)
- added sheet 3_5_RADIO (3_5_RADIO.kicad_sch)
- added sheet 3_6_SD (3_6_SD.kicad_sch)
- note added: "Flash: W25Q128JVE"
- note removed: "0.55 mA"
- note removed: "0.88 mA"
- note removed: "12.5 uA"
- note removed: "15 uA"
- note removed: "500mA"
- note removed: "BARO1: MS5607-02BA03"
- note removed: "BARO2: LPS22HHTR"
- note removed: "IMU1: ICM-42688-P"
- note removed: "IMU2: LSM6DSO32"
- moved on the sheet: BZ401, C403, C404, C407, C410, C411, C412, C413, C414, C415, C416, C417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
