File: 3_1_IMU0.kicad_sch (KiCad schematic)
At the start: 4 parts, among them U601 ICM-42688-P

Commit message: Finished restructuring schematic
Most components that were on page 3 are now in their own page
Added high-frequency 4.7 uF capacitor to servo power line
Continuity sensing on pyrochannels is multiplexed to one ADC on NAV.
Connections:
- net ICM_CS renamed IMU0_CS
- net ICM_INT renamed IMU0_INT
- net ICM_MISO renamed IMU0_MISO
- net ICM_MOSI renamed IMU0_MOSI
- net ICM_SCK renamed IMU0_SCL
Changed lines of the file:
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@@
-	(wire
-		(pts
-			(xy 173.99 90.17) (xy 182.88 90.17)
-		)
-		(stroke
-			(width 0)
-			(type default)
-		)
-	)
 	(wire
 		(pts
@@
 	(wire
 		(pts
-			(xy 123.19 100.33) (xy 132.08 100.33)
-		)
-		(stroke
-			(width 0)
-			(type default)
-		)
-	)
-	(wire
-		(pts
 			(xy 153.67 114.3) (xy 177.8 114.3)
-		)
-		(stroke
-			(width 0)
-			(type default)
-		)
-	)
-	(wire
-		(pts
-			(xy 124.46 95.25) (xy 132.08 95.25)
-		)
-		(stroke
-			(width 0)
-			(type default)
-		)
-	)
-	(wire
-		(pts
-			(xy 123.19 97.79) (xy 132.08 97.79)
 		)
 		(stroke
@@
 	(wire
 		(pts
+			(xy 128.27 102.87) (xy 132.08 102.87)
+		)
+		(stroke
+			(width 0)
+			(type default)
+		)
+	)
+	(wire
+		(pts
 			(xy 109.22 87.63) (xy 111.76 87.63)
+		)
+		(stroke
+			(width 0)
+			(type default)
+		)
+	)
+	(wire
+		(pts
+			(xy 128.27 97.79) (xy 132.08 97.79)
+		)
+		(stroke
+			(width 0)
+			(type default)
+		)
+	)
+	(wire
+		(pts
+			(xy 173.99 90.17) (xy 177.8 90.17)
 		)
 		(stroke
@@
 	(wire
 		(pts
-			(xy 123.19 102.87) (xy 132.08 102.87)
+			(xy 173.99 95.25) (xy 177.8 95.25)
 		)
 		(stroke
@@
 	(wire
 		(pts
-			(xy 173.99 95.25) (xy 177.8 95.25)
+			(xy 128.27 95.25) (xy 132.08 95.25)
 		)
 		(stroke
@@
 		)
 	)
-	(label "ICM_CS"
-		(at 124.46 95.25 0)
+	(wire
+		(pts
+			(xy 128.27 100.33) (xy 132.08 100.33)
+		)
+		(stroke
+			(width 0)
+			(type default)
+		)
+	)
+	(hierarchical_label "IMU0_SCL"
+		(shape input)
+		(at 128.27 97.79 180)
 		(effects
 			(font
 				(size 1.27 1.27)
 			)
-			(justify left bottom)
+			(justify right)
 		)
 	)
-	(label "ICM_MOSI"
-		(at 123.19 100.33 0)
+	(hierarchical_label "IMU0_MISO"
+		(shape output)
+		(at 128.27 102.87 180)
 		(effects
 			(font
 				(size 1.27 1.27)
 			)
-			(justify left bottom)
+			(justify right)
 		)
 	)
-	(label "ICM_SCK"
-		(at 123.19 97.79 0)
+	(hierarchical_label "IMU0_INT"
+		(shape output)
+		(at 177.8 90.17 0)
 		(effects
 			(font
 				(size 1.27 1.27)
 			)
-			(justify left bottom)
+			(justify left)
 		)
 	)
-	(label "ICM_INT"
-		(at 182.88 90.17 180)
+	(hierarchical_label "IMU0_CS"
+		(shape input)
+		(at 128.27 95.25 180)
 		(effects
 			(font
 				(size 1.27 1.27)
 			)
-			(justify right bottom)
+			(justify right)
 		)
 	)
-	(label "ICM_MISO"
-		(at 123.19 102.87 0)
+	(hierarchical_label "IMU0_MOSI"
+		(shape input)
+		(at 128.27 100.33 180)
 		(effects
 			(font
 				(size 1.27 1.27)
 			)
-			(justify left bottom)
+			(justify right)
 		)
 	)
