File: 3_5_RADIO.kicad_sch (KiCad schematic)
At the start: 7 parts, among them J1001 Conn_Coaxial, U1001 Ra-08H

Commit message: Finished restructuring schematic
Most components that were on page 3 are now in their own page
Added high-frequency 4.7 uF capacitor to servo power line
Continuity sensing on pyrochannels is multiplexed to one ADC on NAV.
Changed lines of the file:
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@@
-		)
-	)
-	(label "RF_TX"
-		(at 140.97 101.6 0)
-		(effects
-			(font
-				(size 1.27 1.27)
-			)
-			(justify left bottom)
 		)
 	)
@@
 		)
 	)
-	(label "RF_RX"
-		(at 140.97 99.06 0)
+	(hierarchical_label "RF_RX"
+		(shape input)
+		(at 140.97 99.06 180)
 		(effects
 			(font
 				(size 1.27 1.27)
 			)
-			(justify left bottom)
+			(justify right)
 		)
 	)
+	(hierarchical_label "RF_TX"
+		(shape output)
+		(at 140.97 101.6 180)
+		(effects
+			(font
+				(size 1.27 1.27)
+			)
+			(justify right)
+		)
+	)
