File: polaris.kicad_pcb (KiCad board)
At the start: 4 copper layers, 0 parts

Commit message: Finally started the PCB layout and routing Only took me a few decades Also labeled some unlabeled nets in the schematic Changed the USB mux to be two 1x3 pin headers instead of one 2x3 Edited symbols and footprints to match pin numbers
Parts:
- added BZ401: AC2208, Polaris:AC1255, F.Cu at (200.8, 54.5)
- added C101: 100n, Capacitor_SMD:C_0603_1608Metric, F.Cu at (72.2, 96.4)
- added C102: 100n, Capacitor_SMD:C_0603_1608Metric, F.Cu at (72.2, 98.9)
- added C103: 100n, Capacitor_SMD:C_0603_1608Metric, F.Cu at (72.2, 101.4)
- added C104: 100n, Capacitor_SMD:C_0603_1608Metric, F.Cu at (72.2, 103.9)
- added C201: 100n, Capacitor_SMD:C_0603_1608Metric, F.Cu at (96.8, -39.1)
- added C202: 100n, Capacitor_SMD:C_0603_1608Metric, F.Cu at (96.8, -36.5)
- added C203: 10u, Capacitor_SMD:C_0805_2012Metric, F.Cu at (125.7, -24.6)
- added C204: 4u7, Capacitor_SMD:C_0603_1608Metric, F.Cu at (96.8, -34.0)
- added C205: 10u, Capacitor_SMD:C_0805_2012Metric, F.Cu at (125.7, -21.6)
- added C206: 100n, Capacitor_SMD:C_0603_1608Metric, F.Cu at (96.8, -31.5)
- added C207: 1u, Capacitor_SMD:C_0603_1608Metric, F.Cu at (96.8, -29.0)
- added C208: 1u, Capacitor_SMD:C_0603_1608Metric, F.Cu at (96.8, -26.5)
- added C209: 22u, Capacitor_SMD:C_0805_2012Metric, F.Cu at (125.7, -18.5)
- added C210: 0u22, Capacitor_SMD:C_0603_1608Metric, F.Cu at (96.8, -24.0)
- added C211: 100n, Capacitor_SMD:C_0603_1608Metric, F.Cu at (100.8, -39.1)
- added C212: 4u7, Capacitor_SMD:C_0603_1608Metric, F.Cu at (100.8, -36.5)
- added C213: 10u, Capacitor_SMD:C_0805_2012Metric, F.Cu at (125.7, -15.5)
- added C214: 10u, Capacitor_SMD:C_0805_2012Metric, F.Cu at (125.7, -12.5)
- added C215: 4u7, Capacitor_SMD:C_0603_1608Metric, F.Cu at (100.8, -34.0)
- added C216: 4u7, Capacitor_SMD:C_0603_1608Metric, F.Cu at (100.8, -31.5)
- added C217: 10p, Capacitor_SMD:C_0603_1608Metric, F.Cu at (100.8, -29.0)
- added C301: 100n, Capacitor_SMD:C_0603_1608Metric, F.Cu at (107.8, 153.0)
- added C401: 100n, Capacitor_SMD:C_0603_1608Metric, F.Cu at (169.3, 38.5)
- added C402: 100n, Capacitor_SMD:C_0603_1608Metric, F.Cu at (169.3, 41.0)
- added C403: 100n, Capacitor_SMD:C_0603_1608Metric, F.Cu at (169.3, 43.5)
- added C404: 100n, Capacitor_SMD:C_0603_1608Metric, F.Cu at (169.3, 46.0)
- added C405: 100n, Capacitor_SMD:C_0603_1608Metric, F.Cu at (169.3, 48.5)
- added C406: 100n, Capacitor_SMD:C_0603_1608Metric, F.Cu at (169.3, 51.0)
- added C407: 100n, Capacitor_SMD:C_0603_1608Metric, F.Cu at (169.3, 53.6)
- added C408: 100n, Capacitor_SMD:C_0603_1608Metric, F.Cu at (169.3, 56.1)
- added C409: 4u7, Capacitor_SMD:C_0603_1608Metric, F.Cu at (169.3, 58.6)
- added C410: 100n, Capacitor_SMD:C_0603_1608Metric, F.Cu at (173.3, 38.5)
- added C411: 100n, Capacitor_SMD:C_0603_1608Metric, F.Cu at (173.3, 41.0)
- added C412: 10n, Capacitor_SMD:C_0603_1608Metric, F.Cu at (173.3, 43.5)
- added C413: 100n, Capacitor_SMD:C_0603_1608Metric, F.Cu at (173.3, 46.0)
- added C414: 2u2, Capacitor_SMD:C_0603_1608Metric, F.Cu at (173.3, 48.5)
- added C415: 12p, Capacitor_SMD:C_0603_1608Metric, F.Cu at (173.3, 51.0)
- added C416: 12p, Capacitor_SMD:C_0603_1608Metric, F.Cu at (173.3, 53.6)
- added C417: 12p, Capacitor_SMD:C_0603_1608Metric, F.Cu at (173.3, 56.1)
- added C418: 12p, Capacitor_SMD:C_0603_1608Metric, F.Cu at (173.3, 58.6)
- added C419: 100n, Capacitor_SMD:C_0603_1608Metric, F.Cu at (177.3, 38.5)
- added C501: 100n, Capacitor_SMD:C_0603_1608Metric, F.Cu at (78.7, -39.1)
- added C502: 100n, Capacitor_SMD:C_0603_1608Metric, F.Cu at (78.7, -36.5)
- added C503: 100n, Capacitor_SMD:C_0603_1608Metric, F.Cu at (78.7, -34.0)
- added C504: 100n, Capacitor_SMD:C_0603_1608Metric, F.Cu at (78.7, -31.5)
- added C505: 100n, Capacitor_SMD:C_0603_1608Metric, F.Cu at (78.7, -29.0)
- added C506: 100n, Capacitor_SMD:C_0603_1608Metric, F.Cu at (78.7, -26.5)
- added C507: 100n, Capacitor_SMD:C_0603_1608Metric, F.Cu at (78.7, -24.0)
- added C508: 1u, Capacitor_SMD:C_0603_1608Metric, F.Cu at (82.7, -39.1)
- added C509: 100n, Capacitor_SMD:C_0603_1608Metric, F.Cu at (82.7, -36.5)
- added C510: 100n, Capacitor_SMD:C_0603_1608Metric, F.Cu at (82.7, -34.0)
- added C511: 100n, Capacitor_SMD:C_0603_1608Metric, F.Cu at (82.7, -31.5)
- added C512: 47u, Capacitor_SMD:C_0805_2012Metric, F.Cu at (55.7, 69.5)
- added C513: 10u, Capacitor_SMD:C_0805_2012Metric, F.Cu at (55.7, 72.5)
- added C514: 100n, Capacitor_SMD:C_0603_1608Metric, F.Cu at (82.7, -29.0)
- added C515: 100n, Capacitor_SMD:C_0603_1608Metric, F.Cu at (82.7, -26.5)
- added C601: 2200u, Capacitor_THT:CP_Radial_D13.0mm_P5.00mm, F.Cu at (280.4, 142.5)
- added D201: GREEN, LED_SMD:LED_0603_1608Metric, F.Cu at (123.6, -39.0)
- added D202: ORANGE, LED_SMD:LED_0603_1608Metric, F.Cu at (123.6, -36.4)
- added D301: GREEN, LED_SMD:LED_0603_1608Metric, F.Cu at (120.7, 162.2)
- added D302: ESDS304, Package_TO_SOT_SMD:SOT-23-5, F.Cu at (124.1, 174.3)
- added D303: SMAJ12A, Diode_SMD:D_SMA, F.Cu at (135.1, 173.0)
- added D401: GREEN, LED_SMD:LED_0603_1608Metric, F.Cu at (195.9, 62.7)
- added D402: GREEN, LED_SMD:LED_0603_1608Metric, F.Cu at (195.9, 65.3)
- added D403: GREEN, LED_SMD:LED_0603_1608Metric, F.Cu at (195.9, 67.9)
- added D404: GREEN, LED_SMD:LED_0603_1608Metric, F.Cu at (195.9, 70.5)
- added D501: D_TVS, LED_SMD:LED_0603_1608Metric, F.Cu at (80.7, -12.8)
- added D502: LED, LED_SMD:LED_0603_1608Metric, F.Cu at (80.7, -10.2)
- added D503: LED, LED_SMD:LED_0603_1608Metric, F.Cu at (80.7, -7.57)
- added D504: LED, LED_SMD:LED_0603_1608Metric, F.Cu at (80.7, -4.98)
- added D601: SMAJ9.0CA, Diode_SMD:D_SMA, F.Cu at (279.3, 162.1)
- added H101: MountingHole_Pad, MountingHole:MountingHole_2.5mm_Pad_Via, F.Cu at (67.0, 88.1)
- added H102: MountingHole_Pad, MountingHole:MountingHole_2.5mm_Pad_Via, F.Cu at (67.0, 94.7)
- added H103: MountingHole_Pad, MountingHole:MountingHole_2.5mm_Pad_Via, F.Cu at (67.0, 101.2)
- added H104: MountingHole_Pad, MountingHole:MountingHole_2.5mm_Pad_Via, F.Cu at (67.0, 107.8)
- added J101: XT60-M, Connector_AMASS:AMASS_XT60-F_1x02_P7.20mm_Vertical, F.Cu at (75.4, 90.0)
- added J102: Screw_Terminal_01x02, TerminalBlock:TerminalBlock_Xinya_XY308-2.54-2P_1x02_P2.54mm_Horizontal, F.Cu at (56.0, 80.2)
- added J103: Screw_Terminal_01x02, TerminalBlock:TerminalBlock_Xinya_XY308-2.54-2P_1x02_P2.54mm_Horizontal, F.Cu at (63.7, 80.2)
- added J104: Screw_Terminal_01x02, TerminalBlock:TerminalBlock_Xinya_XY308-2.54-2P_1x02_P2.54mm_Horizontal, F.Cu at (71.3, 80.2)
- added J105: Screw_Terminal_01x02, TerminalBlock:TerminalBlock_Xinya_XY308-2.54-2P_1x02_P2.54mm_Horizontal, F.Cu at (79.0, 80.2)
- added J106: Screw_Terminal_01x02, TerminalBlock:TerminalBlock_Xinya_XY308-2.54-2P_1x02_P2.54mm_Horizontal, F.Cu at (86.6, 80.2)
- added J107: Screw_Terminal_01x02, TerminalBlock:TerminalBlock_Xinya_XY308-2.54-2P_1x02_P2.54mm_Horizontal, F.Cu at (94.2, 80.2)
- added J108: Screw_Terminal_01x03, TerminalBlock:TerminalBlock_Xinya_XY308-2.54-3P_1x03_P2.54mm_Horizontal, F.Cu at (56.0, 89.0)
- added J109: Screw_Terminal_01x03, TerminalBlock:TerminalBlock_Xinya_XY308-2.54-3P_1x03_P2.54mm_Horizontal, F.Cu at (56.0, 97.8)
- added J110: Screw_Terminal_01x03, TerminalBlock:TerminalBlock_Xinya_XY308-2.54-3P_1x03_P2.54mm_Horizontal, F.Cu at (56.0, 106.6)
- added J111: Screw_Terminal_01x03, TerminalBlock:TerminalBlock_Xinya_XY308-2.54-3P_1x03_P2.54mm_Horizontal, F.Cu at (56.0, 115.4)
- added J112: Conn_01x04, Connector_PinHeader_2.00mm:PinHeader_1x04_P2.00mm_Vertical, F.Cu at (89.8, 86.9)
- added J113: Conn_01x04, Connector_PinHeader_2.00mm:PinHeader_1x04_P2.00mm_Vertical, F.Cu at (93.9, 86.9)
- added J114: Screw_Terminal_01x03, TerminalBlock:TerminalBlock_Xinya_XY308-2.54-3P_1x03_P2.54mm_Horizontal, F.Cu at (56.0, 124.2)
- added J301: USB_C_Receptacle_USB2.0_16P, Connector_USB:USB_C_Receptacle_HRO_TYPE-C-31-M-12, F.Cu at (127.2, 184.4)
- added J302: Conn_01x03, Connector_PinHeader_2.54mm:PinHeader_1x03_P2.54mm_Vertical, F.Cu at (67.5, 133.2)
- added J303: Conn_01x03, Connector_PinHeader_2.54mm:PinHeader_1x03_P2.54mm_Vertical, F.Cu at (72.1, 133.2)
- added J401: Screw_Terminal_01x04, TerminalBlock_MetzConnect:TerminalBlock_MetzConnect_Type055_RT01504HDWU_1x04_P5.00mm_Horizontal, F.Cu at (186.8, 42.3)
- added J502: Conn_Coaxial, Connector_Coaxial:SMA_Molex_73251-2200_Horizontal, F.Cu at (58.4, 54.0)
- added J601: XT60-M, Connector_AMASS:AMASS_XT60-F_1x02_P7.20mm_Vertical, F.Cu at (280.4, 130.1)
- added L201: 10u, Inductor_SMD:L_12x12mm_H8mm, F.Cu at (114.2, -33.2)
- added Q201: IRLZ44N, Package_TO_SOT_THT:TO-220-3_Vertical, F.Cu at (110.0, -22.1)
- added Q202: IRLZ44N, Package_TO_SOT_THT:TO-220-3_Vertical, F.Cu at (110.0, -16.2)
- added Q401: Q_NMOS, Package_TO_SOT_SMD:SOT-23, F.Cu at (191.0, 66.9)
- added Q601: IRLZ44N, Package_TO_SOT_THT:TO-220-3_Vertical, F.Cu at (266.9, 128.9)
- added Q602: IRLZ44N, Package_TO_SOT_THT:TO-220-3_Vertical, F.Cu at (266.9, 134.8)
- added Q603: IRLZ44N, Package_TO_SOT_THT:TO-220-3_Vertical, F.Cu at (266.9, 140.8)
- added Q604: IRLZ44N, Package_TO_SOT_THT:TO-220-3_Vertical, F.Cu at (266.9, 146.7)
- added Q605: IRLZ44N, Package_TO_SOT_THT:TO-220-3_Vertical, F.Cu at (266.9, 152.7)
- added Q606: IRLZ44N, Package_TO_SOT_THT:TO-220-3_Vertical, F.Cu at (266.9, 158.6)
- added R201: 360k, Resistor_SMD:R_0603_1608Metric, F.Cu at (100.8, -26.5)
- added R202: 47k, Resistor_SMD:R_0603_1608Metric, F.Cu at (100.8, -24.0)
- added R203: 0R1, Resistor_SMD:R_2512_6332Metric, F.Cu at (111.1, -11.7)
- added R204: 162k, Resistor_SMD:R_0603_1608Metric, F.Cu at (104.8, -39.1)
- added R205: 22.1k, Resistor_SMD:R_0603_1608Metric, F.Cu at (104.8, -36.5)
- added R206: 180R, Resistor_SMD:R_0603_1608Metric, F.Cu at (104.8, -34.0)
- added R207: 180R, Resistor_SMD:R_0603_1608Metric, F.Cu at (104.8, -31.5)
- added R301: 4k7, Resistor_SMD:R_0603_1608Metric, F.Cu at (107.8, 155.5)
- added R302: 180R, Resistor_SMD:R_0603_1608Metric, F.Cu at (107.8, 158.0)
- added R401: 0R, Resistor_SMD:R_0603_1608Metric, F.Cu at (177.3, 41.0)
- added R402: 0R, Resistor_SMD:R_0603_1608Metric, F.Cu at (177.3, 43.5)
- added R403: 4k7, Resistor_SMD:R_0603_1608Metric, F.Cu at (177.3, 46.0)
- added R404: 4k7, Resistor_SMD:R_0603_1608Metric, F.Cu at (177.3, 48.5)
- added R405: 4k7, Resistor_SMD:R_0603_1608Metric, F.Cu at (177.3, 51.0)
- added R406: 4k7, Resistor_SMD:R_0603_1608Metric, F.Cu at (177.3, 53.6)
- added R407: 4k7, Resistor_SMD:R_0603_1608Metric, F.Cu at (177.3, 56.1)
- added R408: 4k7, Resistor_SMD:R_0603_1608Metric, F.Cu at (177.3, 58.6)
- added R409: 180R, Resistor_SMD:R_0603_1608Metric, F.Cu at (181.3, 38.5)
- added R410: 180R, Resistor_SMD:R_0603_1608Metric, F.Cu at (181.3, 41.0)
- added R411: 180R, Resistor_SMD:R_0603_1608Metric, F.Cu at (181.3, 43.5)
- added R412: 180R, Resistor_SMD:R_0603_1608Metric, F.Cu at (181.3, 46.0)
- added R413: 47R, Resistor_SMD:R_0603_1608Metric, F.Cu at (181.3, 48.5)
- added R414: 47k, Resistor_SMD:R_0603_1608Metric, F.Cu at (181.3, 51.0)
- added R501: 27, Resistor_SMD:R_0603_1608Metric, F.Cu at (82.7, -24.0)
- added R502: 27, Resistor_SMD:R_0603_1608Metric, F.Cu at (86.7, -39.1)
- added R503: 1k, Resistor_SMD:R_0603_1608Metric, F.Cu at (86.7, -36.5)
- added R504: 47k, Resistor_SMD:R_0603_1608Metric, F.Cu at (86.7, -34.0)
- added R505: 47k, Resistor_SMD:R_0603_1608Metric, F.Cu at (86.7, -31.5)
- added R506: 47k, Resistor_SMD:R_0603_1608Metric, F.Cu at (86.7, -29.0)
- added R507: 47k, Resistor_SMD:R_0603_1608Metric, F.Cu at (86.7, -26.5)
- added R508: 47k, Resistor_SMD:R_0603_1608Metric, F.Cu at (86.7, -24.0)
- added R509: 180R, Resistor_SMD:R_0603_1608Metric, F.Cu at (90.8, -39.1)
- added R510: 180R, Resistor_SMD:R_0603_1608Metric, F.Cu at (90.8, -36.5)
- added R511: 180R, Resistor_SMD:R_0603_1608Metric, F.Cu at (90.8, -34.0)
- added R512: 10k, Resistor_SMD:R_0603_1608Metric, F.Cu at (90.8, -31.5)
- added R513: 810k, Resistor_SMD:R_0603_1608Metric, F.Cu at (90.8, -29.0)
- added R601: 47R, Resistor_SMD:R_0603_1608Metric, F.Cu at (277.2, 151.0)
- added R602: 47R, Resistor_SMD:R_0603_1608Metric, F.Cu at (277.2, 153.5)
- added R603: 4k7, Resistor_SMD:R_0603_1608Metric, F.Cu at (277.2, 156.0)
- added R604: 4k7, Resistor_SMD:R_0603_1608Metric, F.Cu at (277.2, 158.5)
- added R605: 47R, Resistor_SMD:R_0603_1608Metric, F.Cu at (281.3, 151.0)
- added R606: 47R, Resistor_SMD:R_0603_1608Metric, F.Cu at (281.3, 153.5)
- added R607: 4k7, Resistor_SMD:R_0603_1608Metric, F.Cu at (281.3, 156.0)
- added R608: 4k7, Resistor_SMD:R_0603_1608Metric, F.Cu at (281.3, 158.5)
- added R609: 47R, Resistor_SMD:R_0603_1608Metric, F.Cu at (285.3, 151.0)
- added R610: 47R, Resistor_SMD:R_0603_1608Metric, F.Cu at (285.3, 153.5)
- added R611: 4k7, Resistor_SMD:R_0603_1608Metric, F.Cu at (285.3, 156.0)
- added R612: 4k7, Resistor_SMD:R_0603_1608Metric, F.Cu at (285.3, 158.5)
- added SW401: SW_Push, Button_Switch_THT:SW_PUSH_6mm, F.Cu at (185.3, 49.6)
- added SW402: SW_Push, Button_Switch_THT:SW_PUSH_6mm, F.Cu at (185.3, 58.1)
- added SW501: SW_Push, Button_Switch_THT:SW_PUSH_6mm, F.Cu at (80.6, -20.6)
- added TP501: TestPoint, TestPoint:TestPoint_Pad_2.5x2.5mm, F.Cu at (76.3, -20.3)
- added TP502: TestPoint, TestPoint:TestPoint_Pad_2.5x2.5mm, F.Cu at (76.3, -15.8)
- added TP503: TestPoint, TestPoint:TestPoint_Pad_2.5x2.5mm, F.Cu at (76.3, -11.2)
- added TP504: TestPoint, TestPoint:TestPoint_Pad_2.5x2.5mm, F.Cu at (76.3, -6.67)
- added U201: BQ24005, Package_SO:HTSSOP-20-1EP_4.4x6.5mm_P0.65mm_EP3.4x6.5mm_Mask2.4x3.7mm, F.Cu at (99.6, -10.4)
- added U202: LM74700, Package_TO_SOT_SMD:SOT-23-6, F.Cu at (120.9, -23.7)
- added U203: LM74700, Package_TO_SOT_SMD:SOT-23-6, F.Cu at (120.9, -19.0)
- added U204: NCP1117-3.3, Package_TO_SOT_SMD:SOT-223-3_TabPin2, F.Cu at (99.7, -18.5)
- added U205: LMR51430, Package_TO_SOT_SMD:SOT-23-6, F.Cu at (120.9, -14.4)
- added U206: TPS7A2033PDBVR, Package_TO_SOT_SMD:SOT-23-5, F.Cu at (120.9, -9.79)
- added U301: CH224K, Package_SO:SSOP-10-1EP_3.9x4.9mm_P1mm_EP2.1x3.3mm, F.Cu at (129.4, 167.4)
- added U302: FSUSB42MUX, Package_SO:MSOP-10_3x3mm_P0.5mm, F.Cu at (122.3, 154.1)
- added U401: LPS22HH, Polaris:LPS22HH, F.Cu at (190.4, 71.1)
- added U402: MS5607, Package_LGA:LGA-8_3x5mm_P1.25mm, F.Cu at (205.3, 64.9)
- added U403: STM32F412RGTx, Package_QFP:LQFP-64_10x10mm_P0.5mm, F.Cu at (174.5, 67.1)
- added U404: ICM-42688-P, Polaris:ICM-42688-P, F.Cu at (200.6, 63.4)
- added U405: LSM6DSO32TR, Polaris:LSM6DSO32TR, F.Cu at (200.6, 67.5)
- added U501: W25Q128JVE, Package_SON:WSON-8-1EP_8x6mm_P1.27mm_EP3.4x4.3mm, F.Cu at (87.9, -10.3)
- added U502: RP2040, Package_DFN_QFN:QFN-56-1EP_7x7mm_P0.4mm_EP3.2x3.2mm, F.Cu at (58.5, 63.4)
- added U503: Ra-08H, Polaris:RA-08H, F.Cu at (66.7, -31.5)
- added U504: THD-2528-11SD-GF, Polaris:TF-SMD_THD2528-11SD-GF, F.Cu at (64.9, -15.6)
- added U601: PC817, Package_DIP:DIP-4_W7.62mm, F.Cu at (254.5, 127.0)
- added U602: PC817, Package_DIP:DIP-4_W7.62mm, F.Cu at (254.5, 133.6)
- added U603: PC817, Package_DIP:DIP-4_W7.62mm, F.Cu at (254.5, 140.3)
- added U604: PC817, Package_DIP:DIP-4_W7.62mm, F.Cu at (254.5, 146.9)
- added U605: PC817, Package_DIP:DIP-4_W7.62mm, F.Cu at (254.5, 153.6)
- added U606: PC817, Package_DIP:DIP-4_W7.62mm, F.Cu at (254.5, 160.2)
- added Y401: YXC YSX321SL, Crystal:Crystal_SMD_3225-4Pin_3.2x2.5mm, F.Cu at (185.9, 66.9)
- added Y402: ABRACON ABS05, Crystal:Crystal_SMD_3215-2Pin_3.2x1.5mm, F.Cu at (185.8, 70.9)
Routing:
- net /2_USB/USB_D+: track 0.00 -> 9.15 mm
- net /2_USB/USB_D-: track 0.00 -> 9.12 mm
- net /2_USB/USB_CC2: track 0.00 -> 2.10 mm
- net GND: vias 0 -> 8
- added copper zone on F.Cu, net GND
- added copper zone on In1.Cu, net GND
- added copper zone on In2.Cu, net GND

Commit message: Made an extremely suboptimal ESD protection connection for USB
Parts:
- moved D302 1.86 mm to (125.2, 175.8)
Routing:
- net /2_USB/USB_CC1: track 0.00 -> 10.5 mm
- net /2_USB/USB_D-: track 9.12 -> 13.0 mm
- net /2_USB/USB_D+: track 9.15 -> 12.7 mm
Changed lines of the file:
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@@
 	(footprint "Package_TO_SOT_SMD:SOT-23-5"
 		(layer "F.Cu")
-		(at 124.11 174.35)
+		(at 125.211978 175.846319)
 		(descr "SOT, 5 Pin (JEDEC MO-178 Var AA https://www.jedec.org/document_search?search_api_views_fulltext=MO-178)")
 		(tags "SOT TO_SOT_SMD")
@@
 	)
 	(segment
-		(start 126.782143 174.895877)
-		(end 127.208646 174.895877)
+		(start 125.93 179.64759)
+		(end 124.84241 178.56)
+		(width 0.2)
+		(layer "F.Cu")
+		(net "/2_USB/USB_CC1")
+	)
+	(segment
+		(start 124.84241 178.56)
+		(end 124.83 178.56)
+		(width 0.2)
+		(layer "F.Cu")
+		(net "/2_USB/USB_CC1")
+	)
+	(segment
+		(start 124.83 178.56)
+		(end 124.83 177.99)
+		(width 0.2)
+		(layer "F.Cu")
+		(net "/2_USB/USB_CC1")
+	)
+	(segment
+		(start 123.411979 176.796319)
+		(end 122.29 175.67434)
+		(width 0.2)
+		(layer "F.Cu")
+		(net "/2_USB/USB_CC1")
+	)
+	(segment
+		(start 125.93 180.405)
+		(end 125.93 179.64759)
+		(width 0.2)
+		(layer "F.Cu")
+		(net "/2_USB/USB_CC1")
+	)
+	(segment
+		(start 122.29 175.67434)
+		(end 122.29 171.78)
+		(width 0.2)
+		(layer "F.Cu")
+		(net "/2_USB/USB_CC1")
+	)
+	(segment
+		(start 124.84 177.561841)
+		(end 124.074478 176.796319)
+		(width 0.2)
+		(layer "F.Cu")
+		(net "/2_USB/USB_CC1")
+	)
+	(segment
+		(start 124.074478 176.796319)
+		(end 123.411979 176.796319)
+		(width 0.2)
+		(layer "F.Cu")
+		(net "/2_USB/USB_CC1")
+	)
+	(segment
+		(start 124.83 177.99)
+		(end 124.84 177.98)
+		(width 0.2)
+		(layer "F.Cu")
+		(net "/2_USB/USB_CC1")
+	)
+	(segment
+		(start 124.84 177.98)
+		(end 124.84 177.561841)
+		(width 0.2)
+		(layer "F.Cu")
+		(net "/2_USB/USB_CC1")
+	)
+	(segment
+		(start 125.27 173.876319)
+		(end 125.61 173.536319)
 		(width 0.242062)
 		(layer "F.Cu")
@@
 	)
 	(segment
-		(start 127.208646 174.895877)
-		(end 127.482769 175.17)
+		(start 126.782143 176.672196)
+		(end 127.208646 176.672196)
+		(width 0.242062)
+		(layer "F.Cu")
+		(net "/2_USB/USB_D-")
+	)
+	(segment
+		(start 127.208646 176.672196)
+		(end 127.482769 176.946319)
 		(width 0.242062)
 		(layer "F.Cu")
@@
 	)
 	(segment
+		(start 125.27 176.416319)
+		(end 125.27 173.876319)
+		(width 0.242062)
+		(layer "F.Cu")
+		(net "/2_USB/USB_D-")
+	)
+	(segment
 		(start 127.43 180.405)
 		(end 127.43 179.49)
@@
 	)
 	(segment
+		(start 125.61 172.975247)
+		(end 125.020536 172.385783)
+		(width 0.242062)
+		(layer "F.Cu")
+		(net "/2_USB/USB_D-")
+	)
+	(segment
+		(start 125.65 176.796319)
+		(end 125.27 176.416319)
+		(width 0.242062)
+		(layer "F.Cu")
+		(net "/2_USB/USB_D-")
+	)
+	(segment
 		(start 127.16 179.22)
 		(end 126.71 179.22)
@@
 	)
 	(segment
+		(start 127.482769 179.26473)
+		(end 127.482769 176.970892)
+		(width 0.242062)
+		(layer "F.Cu")
+		(net "/2_USB/USB_D-")
+	)
+	(segment
 		(start 126.71 179.22)
 		(end 126.43 179.5)
@@
 	)
 	(segment
+		(start 125.61 173.536319)
+		(end 125.61 172.975247)
+		(width 0.242062)
+		(layer "F.Cu")
+		(net "/2_USB/USB_D-")
+	)
+	(segment
 		(start 127.43 179.49)
 		(end 127.16 179.22)
@@
 	)
 	(segment
-		(start 127.482769 179.26473)
-		(end 127.482769 175.17)
+		(start 126.349478 176.796319)
+		(end 125.65 176.796319)
 		(width 0.242062)
 		(layer "F.Cu")
@@
 	)
 	(segment
-		(start 127.15 181.53)
-		(end 127.68 181.53)
+		(start 126.339478 173.865797)
+		(end 126.01 173.536319)
 		(width 0.242062)
 		(layer "F.Cu")
@@
 	)
 	(segment
-		(start 127.877231 179.26473)
-		(end 127.877231 175.17)
+		(start 127.93 180.405)
+		(end 127.93 179.317499)
 		(width 0.242062)
 		(layer "F.Cu")
@@
 	)
 	(segment
-		(start 128.682143 174.895877)
-		(end 128.151354 174.895877)
+		(start 127.15 181.53)
+		(end 127.68 181.53)
 		(width 0.242062)
 		(layer "F.Cu")
@@
 	)
 	(segment
-		(start 127.93 180.405)
-		(end 127.93 179.317499)
+		(start 126.349478 174.896319)
+		(end 126.349478 173.865797)
+		(width 0.242062)
+		(layer "F.Cu")
+		(net "/2_USB/USB_D+")
+	)
+	(segment
+		(start 126.01 173.536319)
+		(end 126.01 172.817391)
+		(width 0.242062)
+		(layer "F.Cu")
+		(net "/2_USB/USB_D+")
+	)
+	(segment
+		(start 127.877231 176.818849)
+		(end 127.144701 176.086319)
+		(width 0.242062)
+		(layer "F.Cu")
+		(net "/2_USB/USB_D+")
+	)
+	(segment
+		(start 126.01 172.817391)
+		(end 125.299464 172.106855)
+		(width 0.242062)
+		(layer "F.Cu")
+		(net "/2_USB/USB_D+")
+	)
+	(segment
+		(start 127.144701 176.086319)
+		(end 126.59 176.086319)
 		(width 0.242062)
 		(layer "F.Cu")
@@
 	)
 	(segment
-		(start 128.151354 174.895877)
-		(end 127.877231 175.17)
+		(start 126.349478 175.845797)
+		(end 126.349478 174.896319)
+		(width 0.242062)
+		(layer "F.Cu")
+		(net "/2_USB/USB_D+")
+	)
+	(segment
+		(start 127.877231 179.26473)
+		(end 127.877231 176.818849)
+		(width 0.242062)
+		(layer "F.Cu")
+		(net "/2_USB/USB_D+")
+	)
+	(segment
+		(start 126.59 176.086319)
+		(end 126.349478 175.845797)
 		(width 0.242062)
 		(layer "F.Cu")

Commit message: Continued work on PCB layout
Parts:
- J102: value Screw_Terminal_01x02 -> MAIN1
- J103: value Screw_Terminal_01x02 -> MAIN2
- J104: value Screw_Terminal_01x02 -> MOTOR1
- J105: value Screw_Terminal_01x02 -> MOTOR2
- J106: value Screw_Terminal_01x02 -> DROGUE1
- J107: value Screw_Terminal_01x02 -> DROGUE2
- J108: value Screw_Terminal_01x03 -> FIN1
- J109: value Screw_Terminal_01x03 -> FIN2
- J110: value Screw_Terminal_01x03 -> FIN3
- J111: value Screw_Terminal_01x03 -> FIN4
- J112: value Conn_01x04 -> NAV_SWD
- J113: value Conn_01x04 -> TLM_SWD
- J114: value Screw_Terminal_01x03 -> NAV_GPIO
- J302: value Conn_01x03 -> MUX2
- J303: value Conn_01x03 -> MUX1
- J401: value Screw_Terminal_01x04 -> GNSS
- moved J101 114.8 mm to (179.3, 139.0), turned to -90 degrees
- moved U301 18.8 mm to (112.5, 175.8)
- moved D302 1.17 mm to (125.5, 174.7)
Connections:
- J301 pad SH: SHIELD -> GND
- U504 pad 10: SHIELD -> GND
- U504 pad 11: SHIELD -> GND
- U504 pad 12: SHIELD -> GND
- U504 pad 13: SHIELD -> GND
Routing:
- net /2_USB/USB_CC1: track 10.5 -> 1.41 mm, vias 0 -> 1
- net GND: track 0.00 -> 5.93 mm, vias 8 -> 14
- net /1_Power/USB_VCC: track 0.00 -> 5.64 mm, vias 0 -> 5
- net /2_USB/USB_CC2: track 2.10 -> 1.42 mm, vias 0 -> 1
- net /2_USB/USB_D+: track 12.7 -> 12.2 mm
- added copper zone on F.Cu, net /1_Power/USB_VCC

Commit message: Continued ESD and USB-C section of PCB
Changed ESD device to one more suitable, previously thought unavailable
Started basic component placement
Parts:
- removed D302: ESDS304, Package_TO_SOT_SMD:SOT-23-5
- added U303: USBLC6-2SC6, Package_TO_SOT_SMD:SOT-23-6, F.Cu at (31.3, 126.0)
- added U304: USBLC6-2SC6, Package_TO_SOT_SMD:SOT-23-6, F.Cu at (30.5, 135.2)
- BZ401, Q401, SW401, U504: moved to B.Cu
- moved J601 260.2 mm to (23.1, 91.8), turned to 90 degrees
- moved Q606 174.3 mm to (92.8, 163.9)
- moved Q202 169.2 mm to (73.0, 148.8)
- moved Q201 161.3 mm to (137.8, 136.7)
- moved D303 131.9 mm to (23.1, 103.5)
- moved C601 124.5 mm to (156.1, 149.9)
- moved J301 122.3 mm to (20.0, 125.5), turned to -90 degrees
- moved Y401 118.8 mm to (67.2, 67.1), turned to 180 degrees
- moved J401 115.7 mm to (72.0, 28.2)
- moved Q601 115.3 mm to (159.5, 170.8)
- moved J102 114.9 mm to (110.9, 181.1)
- moved J103 114.9 mm to (118.0, 181.4)
- moved J104 114.3 mm to (125.0, 181.1)
- moved J105 114.3 mm to (132.6, 181.1)
- moved J106 114.3 mm to (140.3, 181.1)
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Connections:
- J301 pad A5: /2_USB/USB_CC1 -> /2_USB/USBC_CC1
- J301 pad A6: /2_USB/USB_D+ -> /2_USB/USBC_D+
- J301 pad A7: /2_USB/USB_D- -> /2_USB/USBC_D-
- J301 pad B5: /2_USB/USB_CC2 -> /2_USB/USBC_CC2
- J301 pad B6: /2_USB/USB_D+ -> /2_USB/USBC_D+
- J301 pad B7: /2_USB/USB_D- -> /2_USB/USBC_D-
Routing:
- net /2_USB/USBC_D+: track 0.00 -> 9.41 mm
- net /2_USB/USBC_D-: track 0.00 -> 7.66 mm
- net GND: track 5.93 -> 10.5 mm, vias 14 -> 20
- net /2_USB/USB_D+: track 12.2 -> 7.93 mm
- net /2_USB/USB_D-: track 12.7 -> 8.57 mm
- net /1_Power/USB_VCC: track 5.64 -> 7.63 mm, vias 5 -> 14
- net /2_USB/USB_CC1: track 1.41 -> 0.00 mm, vias 1 -> 0
- net /TLM_USB_D+: track 0.00 -> 0.84 mm
- net /TLM_USB_D-: track 0.00 -> 0.84 mm
- net /2_USB/USB_CC2: track 1.42 -> 1.95 mm
- added copper zone on B.Cu, net /1_Power/USB_VCC

Commit message: Redesigned the whole thing for the hundredth time
Changed from dual MCU to single MCU
Changed main MCU to STM32F446VE
Added CubeMX project (ioc) file for easy access to pinouts
Note: The PCB file still contains the previous connections and footprints
Parts:
- R413, R414: moved to B.Cu
- moved R605 153.7 mm to (127.6, 152.9), turned to 90 degrees
- moved U601 151.9 mm to (103.3, 141.4)
- moved Q603 141.8 mm to (127.5, 166.9), turned to -90 degrees
- moved Q604 133.4 mm to (135.1, 166.9), turned to -90 degrees
- moved R203 130.8 mm to (37.1, 96.1)
- moved R602 127.2 mm to (150.1, 154.6), turned to 90 degrees
- moved Q605 125.1 mm to (142.6, 166.9), turned to -90 degrees
- moved U603 124.3 mm to (130.2, 139.2), turned to -90 degrees
- moved U504 123.5 mm to (145.9, 63.1), turned to -90 degrees
- moved Q602 121.0 mm to (150.3, 167.0), turned to -90 degrees
- moved U201 114.6 mm to (39.7, 87.4)
- moved U602 102.6 mm to (152.3, 142.4), turned to -90 degrees
- moved SW501 93.5 mm to (128.0, 60.0)
- moved R403 83.7 mm to (87.6, 107.1)
- moved R404 82.9 mm to (87.6, 108.8)
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
Commit message: Began rough component placement
Parts:
- removed C301, C401, C402, C503, C504, C505, C506, C507, C509, C510, C511, C514, C515: 100n, Capacitor_SMD:C_0603_1608Metric
- removed C412: 10n, Capacitor_SMD:C_0603_1608Metric
- removed C508: 1u, Capacitor_SMD:C_0603_1608Metric
- removed C512: 47u, Capacitor_SMD:C_0805_2012Metric
- removed C513: 10u, Capacitor_SMD:C_0805_2012Metric
- removed D303: SMAJ12A, Diode_SMD:D_SMA
- removed D502, D503, D504: LED, LED_SMD:LED_0603_1608Metric
- removed D601: SMAJ9.0CA, Diode_SMD:D_SMA
- removed J302: MUX2, Connector_PinHeader_2.54mm:PinHeader_1x03_P2.54mm_Vertical
- removed J303: MUX1, Connector_PinHeader_2.54mm:PinHeader_1x03_P2.54mm_Vertical
- removed J502: Conn_Coaxial, Connector_Coaxial:SMA_Molex_73251-2200_Horizontal
- removed J601: XT60-M, Connector_AMASS:AMASS_XT60-F_1x02_P7.20mm_Vertical
- removed Q601, Q602, Q603, Q604, Q605, Q606: IRLZ44N, Package_TO_SOT_THT:TO-220-3_Vertical
- removed R302, R410, R411: 180R, Resistor_SMD:R_0603_1608Metric
- removed R401, R402: 0R, Resistor_SMD:R_0603_1608Metric
- removed R403, R404, R603, R604, R607, R608, R611, R612: 4k7, Resistor_SMD:R_0603_1608Metric
- removed R601, R602, R605, R606, R609, R610: 47R, Resistor_SMD:R_0603_1608Metric
- removed SW501: SW_Push, Button_Switch_THT:SW_PUSH_6mm
- removed TP501, TP502, TP503, TP504: TestPoint, TestPoint:TestPoint_Pad_2.5x2.5mm
- removed U304: USBLC6-2SC6, Package_TO_SOT_SMD:SOT-23-6
- removed U401: LPS22HH, Polaris:LPS22HH
- removed U402: MS5607, Package_LGA:LGA-8_3x5mm_P1.25mm
- removed U404: ICM-42688-P, Polaris:ICM-42688-P
- removed U405: LSM6DSO32TR, Polaris:LSM6DSO32TR
- removed U602, U603, U604, U605, U606: PC817, Package_DIP:DIP-4_W7.62mm
- removed Y402: ABRACON ABS05, Crystal:Crystal_SMD_3215-2Pin_3.2x1.5mm
- added C1001: 47u, Capacitor_SMD:C_0805_2012Metric, F.Cu at (99.1, 79.7)
- added C1002: 100n, Capacitor_SMD:C_0603_1608Metric, F.Cu at (94.8, 79.4)
- added C105: 100n, Capacitor_SMD:C_0603_1608Metric, F.Cu at (20.9, 162.0)
- added C106: 100n, Capacitor_SMD:C_0603_1608Metric, F.Cu at (20.9, 164.5)
- added C1101: 10u, Capacitor_SMD:C_0805_2012Metric, B.Cu at (133.7, 71.8)
- added C1102: 100n, Capacitor_SMD:C_0603_1608Metric, B.Cu at (134.1, 79.1)
- added C1201: 100n, Capacitor_SMD:C_0603_1608Metric, F.Cu at (76.5, 92.8)
- added C602: 100n, Capacitor_SMD:C_0603_1608Metric, F.Cu at (126.9, 90.0)
- added C603: 10n, Capacitor_SMD:C_0603_1608Metric, F.Cu at (122.7, 90.7)
- added C701: 100n, Capacitor_SMD:C_0603_1608Metric, F.Cu at (76.5, 97.4)
- added C702: 100n, Capacitor_SMD:C_0603_1608Metric, F.Cu at (76.5, 99.9)
- added C801: 100n, Capacitor_SMD:C_0603_1608Metric, F.Cu at (110.6, 91.5)
- added C901: 100n, Capacitor_SMD:C_0603_1608Metric, F.Cu at (139.9, 88.0)
- added D1001: D_TVS, LED_SMD:LED_0603_1608Metric, F.Cu at (98.9, 82.5)
- added D302: GREEN, LED_SMD:LED_0603_1608Metric, F.Cu at (66.5, 100.4)
- added J1001: Conn_Coaxial, Connector_Coaxial:SMA_Molex_73251-2200_Horizontal, F.Cu at (138.3, 31.4)
- added J115: I2C, TerminalBlock:TerminalBlock_Xinya_XY308-2.54-2P_1x02_P2.54mm_Horizontal, F.Cu at (157.0, 61.8)
- added J116: PB, TerminalBlock:TerminalBlock_Xinya_XY308-2.54-3P_1x03_P2.54mm_Horizontal, F.Cu at (91.1, 52.4)
- added J117: SWD, TerminalBlock:TerminalBlock_Xinya_XY308-2.54-4P_1x04_P2.54mm_Horizontal, F.Cu at (157.1, 55.0)
- added J501: XT60-M, Connector_AMASS:AMASS_XT60-F_1x02_P7.20mm_Vertical, F.Cu at (155.8, 144.6)
- added Q501: IRLZ44N, Package_TO_SOT_THT:TO-220-3_Vertical, F.Cu at (105.4, 158.0)
- added Q502: IRLZ44N, Package_TO_SOT_THT:TO-220-3_Vertical, F.Cu at (105.5, 151.3)
- added Q503: IRLZ44N, Package_TO_SOT_THT:TO-220-3_Vertical, F.Cu at (105.5, 144.7)
- added Q504: IRLZ44N, Package_TO_SOT_THT:TO-220-3_Vertical, F.Cu at (105.5, 138.0)
- added Q505: IRLZ44N, Package_TO_SOT_THT:TO-220-3_Vertical, F.Cu at (105.5, 131.3)
- added Q506: IRLZ44N, Package_TO_SOT_THT:TO-220-3_Vertical, F.Cu at (105.5, 124.6)
- added R1001: 10k, Resistor_SMD:R_0603_1608Metric, F.Cu at (94.8, 81.9)
- added R1002: 810k, Resistor_SMD:R_0603_1608Metric, F.Cu at (94.8, 84.5)
- added R101: 0R, Resistor_SMD:R_0603_1608Metric, F.Cu at (20.9, 167.1)
- added R415: 47k, Resistor_SMD:R_0603_1608Metric, F.Cu at (121.5, 35.8)
- added R514: 47R, Resistor_SMD:R_0603_1608Metric, F.Cu at (110.0, 124.6)
- added R515: 4k7, Resistor_SMD:R_0603_1608Metric, F.Cu at (109.2, 134.0)
- added R516: 4k7, Resistor_SMD:R_0603_1608Metric, F.Cu at (109.2, 127.3)
- added R517: 4k7, Resistor_SMD:R_0603_1608Metric, F.Cu at (68.5, 147.1)
- added R518: 4k7, Resistor_SMD:R_0603_1608Metric, F.Cu at (68.5, 149.6)
- added R519: 1k, Resistor_SMD:R_0603_1608Metric, F.Cu at (68.5, 152.1)
- added R520: 4k7, Resistor_SMD:R_0603_1608Metric, F.Cu at (68.5, 154.7)
- added R801: 4k7, Resistor_SMD:R_0603_1608Metric, F.Cu at (113.9, 84.3)
- added R802: 4k7, Resistor_SMD:R_0603_1608Metric, F.Cu at (108.6, 84.3)
- added R901: 4k7, Resistor_SMD:R_0603_1608Metric, F.Cu at (139.0, 90.4)
- added R902: 4k7, Resistor_SMD:R_0603_1608Metric, F.Cu at (133.3, 88.0)
- added U1001: Ra-08H, Polaris:RA-08H, F.Cu at (143.4, 47.6)
- added U1101: THD-2528-11SD-GF, Polaris:TF-SMD_THD2528-11SD-GF, B.Cu at (151.2, 79.0)
- added U1201: W25Q128JVE, Package_SON:WSON-8-1EP_8x6mm_P1.27mm_EP3.4x4.3mm, B.Cu at (111.1, 57.3)
- added U505: PC817, Package_DIP:DIP-4_W7.62mm, F.Cu at (120.5, 133.9)
- added U506: PC817, Package_DIP:DIP-4_W7.62mm, F.Cu at (120.5, 127.2)
- added U507: CD4051B, Package_SO:SOIC-16_3.9x9.9mm_P1.27mm, F.Cu at (125.6, 117.5)
- added U701: LSM6DSO32TR, Polaris:LSM6DSO32TR, B.Cu at (123.8, 88.4)
- added U801: MS5607, Package_LGA:LGA-8_3x5mm_P1.25mm, F.Cu at (112.5, 88.0)
- added U901: LPS22HH, Polaris:LPS22HH, F.Cu at (137.0, 87.8)
- C201: value 100n -> 0u22
- C202: value 100n -> 10p
- C203: value 10u -> 100n; footprint Capacitor_SMD:C_0805_2012Metric -> Capacitor_SMD:C_0603_1608Metric
- C204, C212: value 4u7 -> 100n
- C205: value 10u -> 4u7; footprint Capacitor_SMD:C_0805_2012Metric -> Capacitor_SMD:C_0603_1608Metric
- C206, C410: value 100n -> 4u7
- C207: value 1u -> 4u7
- C208: value 1u -> 10u; footprint Capacitor_SMD:C_0603_1608Metric -> Capacitor_SMD:C_0805_2012Metric
- C209: value 22u -> 4u7; footprint Capacitor_SMD:C_0805_2012Metric -> Capacitor_SMD:C_0603_1608Metric
- C210: value 0u22 -> 100n
- C211: value 100n -> 10u; footprint Capacitor_SMD:C_0603_1608Metric -> Capacitor_SMD:C_0805_2012Metric
- C213: value 10u -> 1u; footprint Capacitor_SMD:C_0805_2012Metric -> Capacitor_SMD:C_0603_1608Metric
- C215: value 4u7 -> 22u; footprint Capacitor_SMD:C_0603_1608Metric -> Capacitor_SMD:C_0805_2012Metric
- C216: value 4u7 -> 1u
- C217: value 10p -> 10u; footprint Capacitor_SMD:C_0603_1608Metric -> Capacitor_SMD:C_0805_2012Metric
- C403, C404: value 100n -> 12p
- C405: value 100n -> 1u
- C408: value 100n -> 2u2
- C409: value 4u7 -> 2u2
- C414: value 2u2 -> 100n
- C415, C416, C417, C418: value 12p -> 100n
- C501: value 100n -> 2200u; footprint Capacitor_SMD:C_0603_1608Metric -> Capacitor_THT:CP_Radial_D13.0mm_P5.00mm
- C502: value 100n -> C
- C601: value 2200u -> 2u2; footprint Capacitor_THT:CP_Radial_D13.0mm_P5.00mm -> Capacitor_SMD:C_0603_1608Metric
- D301: value GREEN -> SMAJ12A; footprint LED_SMD:LED_0603_1608Metric -> Diode_SMD:D_SMA
- D501: value D_TVS -> SMAJ9.0CA; footprint LED_SMD:LED_0603_1608Metric -> Diode_SMD:D_SMA
- J102: value MAIN1 -> PYRO0
- J103: value MAIN2 -> PYRO1
- J104: value MOTOR1 -> PYRO2
- J105: value MOTOR2 -> PYRO3
- J106: value DROGUE1 -> PYRO4
- J107: value DROGUE2 -> PYRO5
- J108: value FIN1 -> SERVO0
- J109: value FIN2 -> SERVO1
- J110: value FIN3 -> SERVO2
- J111: value FIN4 -> SERVO3
- J112: value NAV_SWD -> SERVO4; footprint Connector_PinHeader_2.00mm:PinHeader_1x04_P2.00mm_Vertical -> TerminalBlock:TerminalBlock_Xinya_XY308-2.54-3P_1x03_P2.54mm_Horizontal
- J113: value TLM_SWD -> SERVO5; footprint Connector_PinHeader_2.00mm:PinHeader_1x04_P2.00mm_Vertical -> TerminalBlock:TerminalBlock_Xinya_XY308-2.54-3P_1x03_P2.54mm_Horizontal
- J114: value NAV_GPIO -> SPI; footprint TerminalBlock:TerminalBlock_Xinya_XY308-2.54-3P_1x03_P2.54mm_Horizontal -> TerminalBlock:TerminalBlock_Xinya_XY308-2.54-4P_1x04_P2.54mm_Horizontal
- J401: footprint TerminalBlock_MetzConnect:TerminalBlock_MetzConnect_Type055_RT01504HDWU_1x04_P5.00mm_Horizontal -> Connector_JST:JST_XH_B4B-XH-A_1x04_P2.50mm_Vertical
- L201: footprint Inductor_SMD:L_12x12mm_H8mm -> Inductor_SMD:L_Sunlord_SWPA8040S
- Q401, SW401: moved to F.Cu
- R204: value 162k -> 180R
- R205: value 22.1k -> 180R
- R206: value 180R -> 162k
- R207: value 180R -> 22.1k
- R301, R408: value 4k7 -> 180R
- R407: value 4k7 -> 0R
- R413: value 47R -> 180R; moved to F.Cu
- R414: value 47k -> 47R; moved to F.Cu
- R501, R502: value 27 -> 47R
- R503: value 1k -> 4k7
- R504, R505, R506: value 47k -> 4k7
- R507, R508: value 47k -> 47R
- R509, R510, R511: value 180R -> 4k7
- R512: value 10k -> 4k7
- R513: value 810k -> 47R
- U204: value NCP1117-3.3 -> TLV75733PDBV; footprint Package_TO_SOT_SMD:SOT-223-3_TabPin2 -> Package_TO_SOT_SMD:SOT-23-5
- U301: value CH224K -> USBLC6-2SC6; footprint Package_SO:SSOP-10-1EP_3.9x4.9mm_P1mm_EP2.1x3.3mm -> Package_TO_SOT_SMD:SOT-23-6
- U302: value FSUSB42MUX -> CH224K; footprint Package_SO:MSOP-10_3x3mm_P0.5mm -> Package_SO:SSOP-10-1EP_3.9x4.9mm_P1mm_EP2.1x3.3mm
- U403: value STM32F412RGTx -> STM32F446VETx; footprint Package_QFP:LQFP-64_10x10mm_P0.5mm -> Package_QFP:LQFP-100_14x14mm_P0.5mm
- U501: value W25Q128JVE -> PC817; footprint Package_SON:WSON-8-1EP_8x6mm_P1.27mm_EP3.4x4.3mm -> Package_DIP:DIP-4_W7.62mm
- U502: value RP2040 -> PC817; footprint Package_DFN_QFN:QFN-56-1EP_7x7mm_P0.4mm_EP3.2x3.2mm -> Package_DIP:DIP-4_W7.62mm
- U503: value Ra-08H -> PC817; footprint Polaris:RA-08H -> Package_DIP:DIP-4_W7.62mm
- U504: value THD-2528-11SD-GF -> PC817; footprint Polaris:TF-SMD_THD2528-11SD-GF -> Package_DIP:DIP-4_W7.62mm; moved to F.Cu
- U601: value PC817 -> ICM-42688-P; footprint Package_DIP:DIP-4_W7.62mm -> Polaris:ICM-42688-P
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Connections:
- C101 pad 1: /5_Pyrochannels/SERVO_PWR -> /4_Pyrochannels/SERVO_PWR
- C101 pad 2: GND -> GND1
- C102 pad 1: /5_Pyrochannels/SERVO_PWR -> /4_Pyrochannels/SERVO_PWR
- C102 pad 2: GND -> GND1
- C103 pad 1: /5_Pyrochannels/SERVO_PWR -> /4_Pyrochannels/SERVO_PWR
- C103 pad 2: GND -> GND1
- C104 pad 1: /5_Pyrochannels/SERVO_PWR -> /4_Pyrochannels/SERVO_PWR
- C104 pad 2: GND -> GND1
- C201 pad 1: VBAT_VIN -> /1_Power/BATT_APG
- C201 pad 2: Net-(U202-VCAP) -> GND
- C202 pad 1: /1_Power/USB_VCC -> Net-(U201-TMR_SEL)
- C202 pad 2: Net-(U203-VCAP) -> GND
- C203 pad 1: +5V -> VBAT_VIN
- C203 pad 2: GND -> Net-(U202-VCAP)
- C204 pad 1: POWER -> /1_Power/USB_VCC
- C204 pad 2: GND -> Net-(U203-VCAP)
- C205 pad 1: +3.3V -> POWER
- C206 pad 1: /1_Power/C_BOOT -> POWER
- C206 pad 2: /1_Power/REG_SW -> GND
- C207 pad 1: +5V -> POWER
- C208 pad 1: +3.3VA -> +5V
- C209 pad 1: +5V -> POWER
- C210 pad 1: /1_Power/BATT_APG -> POWER
- C211 pad 1: POWER -> +3.3V
- C212 pad 1: POWER -> /1_Power/C_BOOT
- C212 pad 2: GND -> /1_Power/REG_SW
- C215 pad 1: POWER -> +5V
- C216 pad 1: POWER -> +3.3VA
- C217 pad 1: Net-(U201-TMR_SEL) -> +5V
- C403 pad 1: +3.3V -> /3_NavigationProcessor/OSC_IN
- C404 pad 1: +3.3V -> /3_NavigationProcessor/OSC_OUT
- C405 pad 1: +3.3V -> Net-(U403-VREF+)
- C406 pad 1: +3.3V -> Net-(U403-VREF+)
- C407 pad 1: +3.3V -> GND
- C407 pad 2: GND -> Net-(U403-NRST)
- C408 pad 1: +3.3V -> Net-(U403-VCAP_1)
- C409 pad 1: +3.3V -> Net-(U403-VCAP_2)
- C415 pad 1: /3_NavigationProcessor/OSC_OUT -> +3.3V
- C416 pad 1: /3_NavigationProcessor/OSC_IN -> +3.3V
- C417 pad 1: /3_NavigationProcessor/RTC_OSC_OUT -> +3.3V
- C418 pad 1: /3_NavigationProcessor/RTC_OSC_IN -> +3.3V
- C419 pad 1: GND -> +3.3V
- C419 pad 2: Net-(U403-NRST) -> GND
- C501 pad 1: +3.3V -> /4_Pyrochannels/SERVO_PWR
- C501 pad 2: GND -> GND1
- C502 pad 1: +3.3V -> /4_Pyrochannels/SERVO_PWR
- C502 pad 2: GND -> GND1
- C601 pad 1: /5_Pyrochannels/SERVO_PWR -> +3.3V
- D301 pad 1: /2_USB/USB_PG -> /1_Power/USB_VCC
- D301 pad 2: Net-(D301-A) -> GND
- D501 pad 1: GND -> GND1
- D501 pad 2: +3.3VA -> /4_Pyrochannels/SERVO_PWR
- J102 pad 2: /5_Pyrochannels/MAIN_1 -> /4_Pyrochannels/PYRO_0
- J103 pad 2: /5_Pyrochannels/MAIN_2 -> /4_Pyrochannels/PYRO_1
- J104 pad 2: /5_Pyrochannels/FIRE_1 -> /4_Pyrochannels/PYRO_2
- J105 pad 2: /5_Pyrochannels/FIRE_2 -> /4_Pyrochannels/PYRO_3
- J106 pad 2: /5_Pyrochannels/DROGUE_1 -> /4_Pyrochannels/PYRO_4
- J107 pad 2: /5_Pyrochannels/DROGUE_2 -> /4_Pyrochannels/PYRO_5
- J108 pad 1: /3_NavigationProcessor/SERVO_S1 -> /3_NavigationProcessor/SERVO_S0
- J108 pad 2: /5_Pyrochannels/SERVO_PWR -> /4_Pyrochannels/SERVO_PWR
- J108 pad 3: GND -> GND1
- J109 pad 1: /3_NavigationProcessor/SERVO_S2 -> /3_NavigationProcessor/SERVO_S1
- J109 pad 2: /5_Pyrochannels/SERVO_PWR -> /4_Pyrochannels/SERVO_PWR
- J109 pad 3: GND -> GND1
- J110 pad 1: /3_NavigationProcessor/SERVO_S3 -> /3_NavigationProcessor/SERVO_S2
- J110 pad 2: /5_Pyrochannels/SERVO_PWR -> /4_Pyrochannels/SERVO_PWR
- J110 pad 3: GND -> GND1
- J111 pad 1: /3_NavigationProcessor/SERVO_S4 -> /3_NavigationProcessor/SERVO_S3
- J111 pad 2: /5_Pyrochannels/SERVO_PWR -> /4_Pyrochannels/SERVO_PWR
- J111 pad 3: GND -> GND1
- J112 pad 1: +3.3V -> /3_NavigationProcessor/SERVO_S4
- J112 pad 2: /3_NavigationProcessor/NAV_SWDIO -> /4_Pyrochannels/SERVO_PWR
- J112 pad 3: /3_NavigationProcessor/NAV_SWCLK -> GND1
- J113 pad 1: GND -> /3_NavigationProcessor/SERVO_S5
- J113 pad 2: /4_TelemetryProcessor/TLM_SWCLK -> /4_Pyrochannels/SERVO_PWR
- J113 pad 3: /4_TelemetryProcessor/TLM_SWDIO -> GND1
- J114 pad 1: /3_NavigationProcessor/NAV_PC10 -> /3_NavigationProcessor/SPI4_SCK
- J114 pad 2: /3_NavigationProcessor/NAV_PC13 -> /3_NavigationProcessor/SPI4_NSS
- J114 pad 3: /3_NavigationProcessor/NAV_ADC1 -> /3_NavigationProcessor/SPI4_MISO
- R204 pad 1: +5V -> Net-(D201-K)
- R204 pad 2: /1_Power/FB -> +3.3V
- R205 pad 1: /1_Power/FB -> Net-(D202-K)
- R205 pad 2: GND -> +3.3V
- R206 pad 1: Net-(D201-K) -> +5V
- R206 pad 2: +3.3V -> /1_Power/FB
- R207 pad 1: Net-(D202-K) -> /1_Power/FB
- R207 pad 2: +3.3V -> GND
- R301 pad 1: /2_USB//MUX_EN -> +3.3V
- R301 pad 2: GND -> Net-(D302-A)
- R405 pad 1: +3.3V -> Net-(U403-BOOT0)
- R405 pad 2: /3_NavigationProcessor/MS_SDA -> GND
- R406 pad 2: /3_NavigationProcessor/MS_SCL -> Net-(U403-NRST)
- R407 pad 1: +3.3V -> /3_NavigationProcessor/OSC_OUT
- R407 pad 2: Net-(U403-NRST) -> Net-(U403-PH1)
- R408 pad 1: Net-(U403-BOOT0) -> /3_NavigationProcessor/NAV_STAT1
- R408 pad 2: GND -> Net-(D401-A)
- R409 pad 1: /3_NavigationProcessor/NAV_STAT1 -> /3_NavigationProcessor/NAV_STAT2
- R409 pad 2: Net-(D403-A) -> Net-(D402-A)
- R412 pad 2: Net-(D402-A) -> Net-(D403-A)
- R413 pad 1: /3_NavigationProcessor/NAV_BUZZ -> /3_NavigationProcessor/NAV_STAT3
- R413 pad 2: Net-(Q401-G) -> Net-(D404-A)
- R414 pad 1: Net-(Q401-G) -> /3_NavigationProcessor/NAV_BUZZ
- R414 pad 2: GND -> Net-(Q401-G)
- R501 pad 1: /TLM_USB_D- -> Net-(Q501-G)
- R501 pad 2: Net-(U502-USB_DM) -> Net-(R501-Pad2)
- R502 pad 1: /TLM_USB_D+ -> Net-(Q502-G)
- R502 pad 2: Net-(U502-USB_DP) -> Net-(R502-Pad2)
- R503 pad 1: /4_TelemetryProcessor/FLASH_SS -> Net-(Q501-G)
- R503 pad 2: Net-(R503-Pad2) -> GND
- R504 pad 1: +3.3V -> Net-(Q502-G)
- R504 pad 2: /4_TelemetryProcessor/SD_CMD -> GND
- R505 pad 1: +3.3V -> /4_Pyrochannels/PYRO_0
- R505 pad 2: /4_TelemetryProcessor/SD_DAT3 -> /4_Pyrochannels/PYRO_0
- R506 pad 1: +3.3V -> /4_Pyrochannels/PYRO_1
- R506 pad 2: /4_TelemetryProcessor/SD_DAT2 -> /4_Pyrochannels/PYRO_1
- R507 pad 1: +3.3V -> Net-(Q503-G)
- R507 pad 2: /4_TelemetryProcessor/SD_DAT1 -> Net-(R507-Pad2)
- R508 pad 1: +3.3V -> Net-(Q504-G)
- R508 pad 2: /4_TelemetryProcessor/SD_DAT0 -> Net-(R508-Pad2)
- R509 pad 1: /4_TelemetryProcessor/TLM_STAT1 -> Net-(Q503-G)
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Routing:
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- removed copper zone on B.Cu, net /1_Power/USB_VCC
- removed copper zone on F.Cu, net /1_Power/USB_VCC
- removed copper zone on F.Cu, net GND
