File: 3_7_FLASH.kicad_sch (KiCad schematic)
At the start: 2 parts, among them U1201 W25Q128JVE

Commit message: Finished most of component re-placement
Began laying tracks for important connections
Parts:
- removed U1201: W25Q128JVE, Package_SON:WSON-8-1EP_8x6mm_P1.27mm_EP3.4x4.3mm, symbol Memory_Flash:W25Q128JVE
- added U1201: W25Q128JVS, Package_SO:SOIC-8_5.3x5.3mm_P1.27mm, symbol Memory_Flash:W25Q128JVS
Connections:
- net +3.3V: now also U1201.8 (VCC)
- net FLASH_CLK: now also U1201.6 (CLK)
- net FLASH_IO0: now also U1201.5 (DI/IO_{0})
- net FLASH_IO1: now also U1201.2 (DO/IO_{1})
- net FLASH_IO2: now also U1201.3 (~{WP}/IO_{2})
- net FLASH_IO3: now also U1201.7 (~{HOLD}/~{RESET}/IO_{3})
- net GND: now also U1201.4 (GND)
- net ~{FLASH_CS}: now also U1201.1 (~{CS})
Changed lines of the file:
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@@
 	(paper "A4")
-	(junction
-		(at 144.78 120.65)
-		(diameter 0)
-		(color 0 0 0 0)
-	)
 	(junction
 		(at 144.78 90.17)
@@
 		(pts
 			(xy 154.94 105.41) (xy 158.75 105.41)
-		)
-		(stroke
-			(width 0)
-			(type default)
-		)
-	)
-	(wire
-		(pts
-			(xy 142.24 120.65) (xy 144.78 120.65)
 		)
 		(stroke
@@
 	)
 	(symbol
-		(lib_id "Memory_Flash:W25Q128JVE")
+		(lib_id "Memory_Flash:W25Q128JVS")
 		(at 144.78 107.95 0)
 		(mirror y)
@@
 		(in_pos_files yes)
 		(dnp no)
+		(fields_autoplaced yes)
 		(property "Reference" "U1201"
-			(at 132.842 106.6799 0)
+			(at 133.35 106.6799 0)
 			(show_name no)
 			(do_not_autoplace no)
@@
 			)
 		)
-		(property "Value" "W25Q128JVE"
-			(at 132.842 109.2199 0)
+		(property "Value" "W25Q128JVS"
+			(at 133.35 109.2199 0)
 			(show_name no)
 			(do_not_autoplace no)
@@
 			)
 		)
-		(property "Footprint" "Package_SON:WSON-8-1EP_8x6mm_P1.27mm_EP3.4x4.3mm"
+		(property "Footprint" "Package_SO:SOIC-8_5.3x5.3mm_P1.27mm"
 			(at 144.78 85.09 0)
 			(hide yes)
@@
 			)
 		)
-		(property "Description" "128Mbit / 16MiB Serial Flash Memory, Standard/Dual/Quad SPI, 2.7-3.6V, WSON-8"
+		(property "Description" "128Mbit / 16MiB Serial Flash Memory, Standard/Dual/Quad SPI, 2.7-3.6V, SOIC-8"
 			(at 144.78 80.01 0)
 			(hide yes)
@@
 			)
 		)
-		(property "Description_1" ""
-			(at 144.78 107.95 0)
-			(hide yes)
-			(show_name no)
-			(do_not_autoplace no)
-			(effects
-				(font
-					(size 1.27 1.27)
-				)
-			)
-		)
-		(property "KLC_S3.3" ""
-			(at 144.78 107.95 0)
-			(hide yes)
-			(show_name no)
-			(do_not_autoplace no)
-			(effects
-				(font
-					(size 1.27 1.27)
-				)
-			)
-		)
-		(property "KLC_S4.1" ""
-			(at 144.78 107.95 0)
-			(hide yes)
-			(show_name no)
-			(do_not_autoplace no)
-			(effects
-				(font
-					(size 1.27 1.27)
-				)
-			)
-		)
-		(property "KLC_S4.2_DVDD" ""
-			(at 144.78 107.95 0)
-			(hide yes)
-			(show_name no)
-			(do_not_autoplace no)
-			(effects
-				(font
-					(size 1.27 1.27)
-				)
-			)
-		)
-		(property "KLC_S4.2_VREG_VOUT" ""
-			(at 144.78 107.95 0)
-			(hide yes)
-			(show_name no)
-			(do_not_autoplace no)
-			(effects
-				(font
-					(size 1.27 1.27)
-				)
-			)
-		)
-		(property "LCSC Part Name" ""
-			(at 144.78 107.95 0)
-			(hide yes)
-			(show_name no)
-			(do_not_autoplace no)
-			(effects
-				(font
-					(size 1.27 1.27)
-				)
-			)
-		)
-		(property "Manufacturer Part" ""
-			(at 144.78 107.95 0)
-			(hide yes)
-			(show_name no)
-			(do_not_autoplace no)
-			(effects
-				(font
-					(size 1.27 1.27)
-				)
-			)
-		)
-		(property "Supplier" ""
-			(at 144.78 107.95 0)
-			(hide yes)
-			(show_name no)
-			(do_not_autoplace no)
-			(effects
-				(font
-					(size 1.27 1.27)
-				)
-			)
-		)
-		(property "Supplier Part" ""
-			(at 144.78 107.95 0)
-			(hide yes)
-			(show_name no)
-			(do_not_autoplace no)
-			(effects
-				(font
-					(size 1.27 1.27)
-				)
-			)
+		(pin "3"
+		)
+		(pin "2"
 		)
 		(pin "1"
 		)
+		(pin "7"
+		)
+		(pin "6"
+		)
 		(pin "4"
 		)
-		(pin "6"
-		)
 		(pin "8"
 		)
-		(pin "7"
-		)
-		(pin "9"
-		)
-		(pin "2"
-		)
-		(pin "3"
-		)
 		(pin "5"
