File: 4_Pyro.kicad_sch (KiCad schematic)
At the start: 37 parts, among them J501 XT60-M, Q501 IRLZ44N, Q502 IRLZ44N, Q503 IRLZ44N, Q504 IRLZ44N, Q505 IRLZ44N, Q506 IRLZ44N, U501 PC817, U502 PC817, U503 CD4051B, U504 PC817, U505 PC817, U506 PC817, U507 PC817

Commit message: Revised schematic for easier routing
Parts:
- C502: footprint Capacitor_SMD:C_0603_1608Metric -> Capacitor_SMD:C_0805_2012Metric
Connections:
- net PYRO_C4: now also U503.1 (X4); no longer U503.5 (X5)
- net PYRO_C5: now also U503.5 (X5); no longer U503.1 (X4)
Changed lines of the file:
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@@
 		)
 	)
-	(label "PYRO_C5"
+	(label "PYRO_C4"
 		(at 44.45 153.67 0)
 		(effects
@@
 		)
 	)
-	(label "PYRO_C4"
+	(label "PYRO_C5"
 		(at 44.45 156.21 0)
 		(effects
@@
 			)
 		)
-		(property "Footprint" "Capacitor_SMD:C_0603_1608Metric"
+		(property "Footprint" "Capacitor_SMD:C_0805_2012Metric"
 			(at 215.5952 156.21 0)
 			(hide yes)
