File: 3_4_BARO1.kicad_sch (KiCad schematic)
At the start: 4 parts, among them U901 LPS22HH

Commit message: Completed PCB
Added logo because why not
Added fillets to corners
Parts:
- U901: footprint Polaris:LPS22HH -> Package_LGA:ST_HLGA-10_2x2mm_P0.5mm_LayoutBorder3x2y
Changed lines of the file:
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@@
 			)
 		)
-		(property "Footprint" "Polaris:LPS22HH"
+		(property "Footprint" "Package_LGA:ST_HLGA-10_2x2mm_P0.5mm_LayoutBorder3x2y"
 			(at 140.97 111.76 0)
 			(hide yes)
